Commit message: update URDF parameters

File: src/nova_description/urdf/nova.urdf.xacro (robot description, xacro)
@@ -90,11 +90,11 @@
     <axis xyz="0.0 1.0 0.0"/>
   </joint>
-  <!-- MPU6050 -->
+  <!-- MPU6050
   <link name="imu_link"/>
   <joint name="imu_joint" type="fixed">
-    <origin xyz="0.05 0 0.25" rpy="0 0 0"/>
+    <origin xyz="0.0 0.0 0.0" rpy="0 0 0"/>
     <parent link="base_link"/>
     <child link="imu_link"/>
-  </joint>
+  </joint> -->
   <link name="Raspberry_pi_4_case">
       <inertial>
